File: design/centauri.kicad_pcb (KiCad board)
At the start: 2 copper layers, 28.2 x 71.2 mm, 66 parts, among them J1 USB_C_Receptacle_USB2.0_14P, J2 Conn_01x28, J3 Conn_01x28, SW1 SW_Push, SW2 SW_Push, U1 PCM5102A, U2 IP5306, U3 RP2354B, U4 XC6206PxxxMR, Y1 Crystal_GND24

Commit message: Fixed PCB and Gerber files
Routing:
- net GND: track 181.3 -> 249.0 mm, vias 22 -> 30
- net +3V3: track 101.2 -> 155.2 mm, vias 1 -> 3
- net GP11: track 18.4 -> 19.4 mm
- net VREG_LX: track 8.88 -> 9.88 mm
- net SWCLK: track 24.9 -> 25.7 mm
- net GP10: track 20.8 -> 21.5 mm
- net GP19: track 21.5 -> 21.0 mm

Commit message: Fixed PCB and README.md images
Parts:
- moved C14 20.0 mm to (248.8, 63.3), turned to 45 degrees
- moved C7 19.2 mm to (239.4, 56.7), turned to 180 degrees
- moved C8 16.8 mm to (239.4, 57.8), turned to 180 degrees
- moved C12 14.8 mm to (252.1, 71.0), turned to 45 degrees
- moved C6 14.4 mm to (239.4, 58.9), turned to 180 degrees
- moved C18 13.9 mm to (251.3, 70.2), turned to 45 degrees
- moved C31 12.8 mm to (238.9, 98.1), turned to -90 degrees
- moved C15 12.0 mm to (247.7, 74.2), turned to -45 degrees
- moved C27 10.1 mm to (248.2, 90.4)
- moved C32 8.46 mm to (239.9, 90.5)
- moved C17 8.41 mm to (246.8, 75.0), turned to -45 degrees
- moved C30 6.49 mm to (248.8, 92.5), turned to -90 degrees
- moved C1 6.48 mm to (245.9, 60.5), turned to 45 degrees
- moved C29 5.45 mm to (247.1, 90.4)
- moved C13 5.35 mm to (239.0, 72.8), turned to -135 degrees
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Routing:
- net GND: track 249.0 -> 123.4 mm, vias 30 -> 29
- net VREG_FB: track 27.5 -> 9.87 mm
- net GP37: track 51.3 -> 33.8 mm, vias 0 -> 2
- net Net-(U3-RUN): track 36.7 -> 51.5 mm, vias 4 -> 2
- net SWCLK: track 25.7 -> 13.5 mm, vias 4 -> 1
- net ADC5: track 18.6 -> 29.3 mm, vias 1 -> 2
- net ADC7: track 25.6 -> 35.6 mm, vias 1 -> 3
- net GP36: track 44.0 -> 34.3 mm, vias 0 -> 2
- net Net-(U2-BAT): track 32.3 -> 23.2 mm
- net ADC4: track 16.1 -> 24.8 mm, vias 1 -> 2
- net Net-(R6-Pad1): track 19.7 -> 28.4 mm
- net GP38: track 43.8 -> 35.3 mm
- net ADC6: track 24.1 -> 31.9 mm, vias 1 -> 2
- net GP26: track 34.0 -> 41.7 mm
- net +3V3: track 155.2 -> 162.2 mm, vias 3 -> 18
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- added copper zone on In1.Cu, net GND
- removed copper zone on F.Cu, net GND
Other:
- copper layers 2 -> 4
